File: HW/IR_lights.kicad_pcb (KiCad board)
At the start: 2 copper layers, 60.2 x 19.8 mm, 29 parts, among them J1 Conn_02x05_Odd_Even, J2 Conn_01x04, J3 Conn_01x02, SW1 SW_Push_Dual, SW2 SW_Push_Dual, SW3 SW_Push_Dual, U1 ATSAMD21E15L-M, U2 ATSAMD21E15L-A

Commit message: Oprava proudu do IR lekdy + SDA,SDC
Parts:
- added Q1: 2N7002H, Package_TO_SOT_SMD:SOT-23, F.Cu at (158.0, 100.4)
- moved R9 7.98 mm to (153.3, 108.4), turned to 180 degrees
- moved D4 2.60 mm to (185.9, 101.4), turned to -90 degrees
Connections:
- D4 pad 1: GND -> Net-(D4-Pad1)
- R9 pad 1: /IR_TRANSMITTER -> Net-(D4-Pad2)
- R9 pad 2: Net-(D4-Pad2) -> +3V3
- U1 pad 17: /SCL -> /SDA
- U1 pad 18: /SDA -> /SCL
- U2 pad 17: /SCL -> /SDA
- U2 pad 18: /SDA -> /SCL
Routing:
- net Net-(D4-Pad1): track 0.00 -> 27.4 mm
- net /SCL: track 22.7 -> 18.6 mm
- net Net-(D4-Pad2): track 30.6 -> 34.4 mm
- net +3V3: track 57.7 -> 58.7 mm
- net /IR_TRANSMITTER: track 4.76 -> 5.49 mm
- net /SDA: track 17.5 -> 18.1 mm
- net GND: vias 17 -> 21

Commit message: Zmena otvoru pro uchyceni modulu
Parts:
- J2: footprint Connector_PinHeader_2.54mm:PinHeader_1x04_P2.54mm_Vertical -> Connector_PinHeader_2.54mm:PinHeader_1x04_P2.54mm_Horizontal
- J3: footprint Connector_PinSocket_2.54mm:PinSocket_1x02_P2.54mm_Vertical -> Connector_PinHeader_2.54mm:PinHeader_1x02_P2.54mm_Vertical
- moved J2 2.50 mm to (134.0, 106.2)
Routing:
- net GND: track 31.7 -> 37.0 mm
- net /SDA: track 18.1 -> 15.5 mm
- net /SCL: track 18.6 -> 16.1 mm
- net +3V3: track 58.7 -> 57.7 mm
- net (no net): vias 0 -> 1
