File: HW/IR_lights.kicad_sch (KiCad schematic)
At the start: 29 parts, among them J1 Conn_02x05_Odd_Even, J2 Conn_01x04, J3 Conn_01x02, SW1 SW_Push_Dual, SW2 SW_Push_Dual, SW3 SW_Push_Dual, U1 ATSAMD21E15L-M, U2 ATSAMD21E15L-A

Commit message: Oprava proudu do IR lekdy + SDA,SDC
Parts:
- removed C8: 0.1uF, Capacitor_SMD:C_0402_1005Metric, symbol Device:C
- added Q1: 2N7002H, Package_TO_SOT_SMD:SOT-23, symbol Transistor_FET:2N7002H
Connections:
- net +3V3: now also R9.2
- net GND: now also Q1.2 (S); no longer D4.1 (K)
- net IR_TRANSMITTER: now also Q1.1 (G); no longer R9.1
- net SCL: now also U1.18 (PA17), U2.18 (PA17); no longer U1.17 (PA16), U2.17 (PA16)
- net SDA: now also U1.17 (PA16), U2.17 (PA16); no longer U1.18 (PA17), U2.18 (PA17)
- net at D4.2 (A): now also R9.1; no longer R9.2
- new net: D4.1 (K), Q1.3 (D)
Other:
- moved on the sheet: D4, R9

Commit message: Zmena otvoru pro uchyceni modulu
Parts:
- J2: footprint Connector_PinHeader_2.54mm:PinHeader_1x04_P2.54mm_Vertical -> Connector_PinHeader_2.54mm:PinHeader_1x04_P2.54mm_Horizontal
- J3: footprint Connector_PinSocket_2.54mm:PinSocket_1x02_P2.54mm_Vertical -> Connector_PinHeader_2.54mm:PinHeader_1x02_P2.54mm_Vertical
Changed lines of the file:
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@@
       (effects (font (size 1.27 1.27)) (justify left))
     )
-    (property "Footprint" "Connector_PinHeader_2.54mm:PinHeader_1x04_P2.54mm_Vertical" (id 2) (at 185.42 148.59 0)
+    (property "Footprint" "Connector_PinHeader_2.54mm:PinHeader_1x04_P2.54mm_Horizontal" (id 2) (at 185.42 148.59 0)
       (effects (font (size 1.27 1.27)) hide)
     )
@@
       (effects (font (size 1.27 1.27)) (justify left))
     )
-    (property "Footprint" "Connector_PinSocket_2.54mm:PinSocket_1x02_P2.54mm_Vertical" (id 2) (at 224.79 148.59 0)
+    (property "Footprint" "Connector_PinHeader_2.54mm:PinHeader_1x02_P2.54mm_Vertical" (id 2) (at 224.79 148.59 0)
       (effects (font (size 1.27 1.27)) hide)
     )
@@
     )
     (path "/a502b8c2-03f0-4066-a20f-b7cf7699e3cd"
-      (reference "J2") (unit 1) (value "Conn_01x04") (footprint "Connector_PinHeader_2.54mm:PinHeader_1x04_P2.54mm_Vertical")
+      (reference "J2") (unit 1) (value "Conn_01x04") (footprint "Connector_PinHeader_2.54mm:PinHeader_1x04_P2.54mm_Horizontal")
     )
     (path "/d898f9b8-51e8-441d-a2c3-5781b195ce2f"
-      (reference "J3") (unit 1) (value "Conn_01x02") (footprint "Connector_PinSocket_2.54mm:PinSocket_1x02_P2.54mm_Vertical")
+      (reference "J3") (unit 1) (value "Conn_01x02") (footprint "Connector_PinHeader_2.54mm:PinHeader_1x02_P2.54mm_Vertical")
     )
     (path "/987f0bd7-7b14-4571-8926-3fb01fef165e"
